Commit message: gazebo wheel state update

File: turtlebot3/turtlebot3_description/urdf/turtlebot3_burger.gazebo.xacro (robot description, xacro)
@@ -58,5 +58,5 @@
       <rightJoint>wheel_right_joint</rightJoint>
       <wheelSeparation>0.160</wheelSeparation>
-      <wheelDiameter>0.066</wheelDiameter>
+      <wheelDiameter>0.110</wheelDiameter>
       <wheelAcceleration>1</wheelAcceleration>
       <wheelTorque>10</wheelTorque>

File: turtlebot3/turtlebot3_description/urdf/turtlebot3_burger_for_autorace.urdf.xacro (robot description, xacro)
@@ -48,5 +48,5 @@
       <origin xyz="0 0 0" rpy="0 0 0"/>
       <geometry>
-        <cylinder length="0.018" radius="0.033"/>
+        <cylinder length="0.018" radius="0.055"/>
       </geometry>
     </collision>
@@ -76,5 +76,5 @@
       <origin xyz="0 0 0" rpy="0 0 0"/>
       <geometry>
-        <cylinder length="0.018" radius="0.033"/>
+        <cylinder length="0.018" radius="0.055"/>
       </geometry>
     </collision>
@@ -129,5 +129,5 @@
       <origin xyz="0.015 0 -0.0065" rpy="0 0 0"/>
       <geometry>
-        <cylinder length="0.0315" radius="0.055"/>
+        <cylinder length="0.0315" radius="0.033"/>
       </geometry>
     </collision>

File: turtlebot3/turtlebot3_description/urdf/turtlebot3_burger_for_autorace_2020.gazebo.xacro (robot description, xacro)
@@ -59,5 +59,5 @@
       <rightJoint>wheel_right_joint</rightJoint>
       <wheelSeparation>0.160</wheelSeparation>
-      <wheelDiameter>0.066</wheelDiameter>
+      <wheelDiameter>0.110</wheelDiameter>
       <wheelAcceleration>1</wheelAcceleration>
       <wheelTorque>10</wheelTorque>
