Commit message: gazebo lidar yaw setting

File: turtlebot3/turtlebot3_description/urdf/turtlebot3_burger_for_autorace_2020.urdf.xacro (robot description, xacro)
@@ -116,9 +116,9 @@
     <parent link="base_link"/>
     <child link="base_scan"/>
-    <origin xyz="-0.032 0 0.172" rpy="0 0 0"/>
+    <origin xyz="-0.032 0 0.172" rpy="0 0 3.14"/>
   </joint>
   <link name="base_scan">
     <visual>
-      <origin xyz="0 0 0.0" rpy="0 0 0"/>
+      <origin xyz="0 0 0.0" rpy="0 0 3.14"/>
       <geometry>
         <mesh filename="package://turtlebot3_description/meshes/sensors/lds.stl" scale="0.001 0.001 0.001"/>
@@ -127,5 +127,5 @@
     </visual>
     <collision>
-      <origin xyz="0.015 0 -0.0065" rpy="0 0 0"/>
+      <origin xyz="0.015 0 -0.0065" rpy="0 0 3.14"/>
       <geometry>
         <cylinder length="0.0315" radius="0.055"/>
